Commit message: Add Distance sensor
Enable show distance sensor ray by default on webots

File: resource/urdf/Assemblage_Carcasse.urdf (robot description, URDF)
Before this commit: robot Assemblage_Carcasse, 9 links, 8 joints
Links:
- added link range_meter_link, mass 0.000523598775598299; visual sphere radius=0.01
Joints:
- added joint range_meter_joint: type fixed, parent base_link, child range_meter_link, origin xyz=0.1 -0.10799191350927 0.2 rpy=0 0 0, axis 0 0 0
