Commit message: Added robot to CDR_2026 world
Modified arena floor to allow jpg to work with webots and ros2 launch

File: resource/Robot/urdf/Assemblage_Carcasse.urdf (robot description, URDF)
Before this commit: robot Assemblage_Carcasse, 11 links, 10 joints
Links:
- link arm_left_link: geometry collision mesh filename=package://simulateur_robot_2016/resource/Robot/meshes/colli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; visual mesh filename=package://simulateur_robot_2016/resource/Robot/meshes/visua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
- link arm_right_link: geometry collision mesh filename=package://simulateur_robot_2016/resource/Robot/meshes/colli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; visual mesh filename=package://simulateur_robot_2016/resource/Robot/meshes/visua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
- link base_link: geometry collision mesh filename=package://simulateur_robot_2016/resource/Robot/meshes/colli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; visual mesh filename=package://simulateur_robot_2016/resource/Robot/meshes/visua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

Commit message: Modified box collision for arms
Updated URDF

File: resource/Robot/urdf/Assemblage_Carcasse.urdf (robot description, URDF)
Before this commit: robot Assemblage_Carcasse, 11 links, 10 joints
Links:
- link arm_left_link: geometry collision box size=0.12 0.006 0.08; visual mesh filename=package://simulateur_robot_2016/resource/Robot/meshes/visua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
- link arm_right_link: geometry collision box size=0.12 0.006 0.08; visual mesh filename=package://simulateur_robot_2016/resource/Robot/meshes/visua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
